File: Hardware/Moisture_Sensor/Moisture Sensor.kicad_pcb (KiCad board)
At the start: 2 copper layers, 135.4 x 28.4 mm, 26 parts, among them J1 Conn_01x02_Pin, J2 Conn_01x02_Pin, J3 Conn_01x03_Pin, Q1 BSS123, Q2 BSS84, U1 ESP32-H2-SUPERMINI, U3 NE555D

Commit message: layout angepasst. dokumentation hinzugefügt
Parts:
- moved G*** 2.55 mm to (130.0, 87.9)
Routing:
- net GND: track 19.3 -> 32.1 mm, vias 14 -> 35
- net Net-(D1-A): track 91.3 -> 89.8 mm
Other:
- board text added: "Moisture Sensor (OpenThread) V 1.0 - 04.2026"
