File: Hardware/Moisture_Sensor/Moisture Sensor.kicad_pcb (KiCad board)
At the start: 2 copper layers, 135.4 x 28.4 mm, 26 parts, among them J1 Conn_01x02_Pin, J2 Conn_01x02_Pin, J3 Conn_01x03_Pin, Q1 BSS123, Q2 BSS84, U1 ESP32-H2-SUPERMINI, U3 NE555D

Commit message: R2 auf 330 geändert und R5 auf 1Meg
Parts:
- removed REF**: 3.7V 500mAh, Lithium:3.7V 500mAh
- R2: value 330k -> 330
- R5: value 10k -> 1M
Changed lines of the file:
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@@
 		(sheetname "/")
 		(sheetfile "Moisture Sensor.kicad_sch")
-		(attr through_hole exclude_from_bom dnp)
+		(attr through_hole exclude_from_bom)
 		(fp_line
 			(start -1.38 6.46)
@@
 			)
 		)
-		(property "Value" "10k"
+		(property "Value" "1M"
 			(at 0 1.43 0)
 			(layer "F.Fab")
@@
 		(sheetname "/")
 		(sheetfile "Moisture Sensor.kicad_sch")
-		(attr through_hole exclude_from_bom dnp)
+		(attr through_hole)
 		(fp_line
 			(start -1.38 -1.38)
@@
 		(sheetname "/")
 		(sheetfile "Moisture Sensor.kicad_sch")
-		(attr through_hole exclude_from_bom dnp)
+		(attr through_hole)
 		(fp_line
 			(start -1.38 3.92)
@@
 			(effects
 				(font
-					(size 0.5 0.5)
+					(size 1 1)
 					(thickness 0.1)
 					(bold yes)
@@
 			)
 		)
-		(property "Value" "330k"
+		(property "Value" "330"
 			(at 0 1.43 0)
 			(layer "F.Fab")
@@
 		)
 	)
-	(footprint "Lithium:3.7V 500mAh"
-		(layer "B.Cu")
-		(at 170.688 87.63 180)
-		(property "Reference" "REF**"
-			(at 0.254 9.12 0)
-			(unlocked yes)
-			(layer "B.SilkS")
-			(effects
-				(font
-					(size 1 1)
-					(thickness 0.1)
-				)
-				(justify mirror)
-			)
-		)
-		(property "Value" "3.7V 500mAh"
-			(at 0.254 7.62 0)
-			(unlocked yes)
-			(layer "B.Fab")
-			(effects
-				(font
-					(size 1 1)
-					(thickness 0.15)
-				)
-				(justify mirror)
-			)
-		)
-		(property "Datasheet" ""
-			(at 0 0 0)
-			(unlocked yes)
-			(layer "B.Fab")
-			(hide yes)
-			(effects
-				(font
-					(size 1 1)
-					(thickness 0.15)
-				)
-				(justify mirror)
-			)
-		)
-		(property "Description" ""
-			(at 0 0 0)
-			(unlocked yes)
-			(layer "B.Fab")
-			(hide yes)
-			(effects
-				(font
-					(size 1 1)
-					(thickness 0.15)
-				)
-				(justify mirror)
-			)
-		)
-		(attr smd)
-		(fp_rect
-			(start 20.828 12.446)
-			(end 21.844 5.842)
-			(stroke
-				(width 0.1)
-				(type default)
-			)
-			(fill no)
-			(layer "B.SilkS")
-		)
-		(fp_rect
-			(start -14.986 12.47)
-			(end 20.828 -12.422)
-			(stroke
-				(width 0.1)
-				(type default)
-			)
-			(fill no)
-			(layer "B.SilkS")
-		)
-		(fp_text user "${REFERENCE}"
-			(at 0.254 6.12 0)
-			(unlocked yes)
-			(layer "B.Fab")
-			(effects
-				(font
-					(size 1 1)
-					(thickness 0.15)
-				)
-				(justify mirror)
-			)
-		)
-		(embedded_fonts no)
-		(model "${KIPRJMOD}/Lithium.pretty/3.7v li-ion 500mah Battery.step"
-			(offset
-				(xyz 3.5 0 -2)
-			)
-			(scale
-				(xyz 1 1 1)
-			)
-			(rotate
-				(xyz -90 -0 -90)
-			)
-		)
-	)
 	(gr_line
 		(start 62.619489 97.791391)
@@
 	)
 	(zone
-		(net 32)
-		(net_name "IO4")
-		(layer "F.Cu")
-		(name "$teardrop_padvia$")
-		(hatch none 0.1)
-		(priority 30002)
-		(attr
-			(teardrop
-				(type padvia)
-			)
-		)
-		(connect_pads yes
-			(clearance 0)
-		)
-		(min_thickness 0.0254)
-		(filled_areas_thickness no)
-		(fill yes
-			(thermal_gap 0.5)
-			(thermal_bridge_width 0.5)
-			(island_removal_mode 1)
-			(island_area_min 10)
-		)
-		(polygon
-			(pts
-				(xy 169.264 76.974169) (xy 169.064 76.974169) (xy 168.531075 78.04308) (xy 169.154677 79.910758)
-				(xy 169.778279 78.04308)
-			)
-		)
-	)
-	(zone
 		(net 29)
 		(net_name "Net-(U1-IO11)")
@@
 			)
 		)
-	)
-	(zone
-		(net 31)
-		(net_name "IO5")
-		(layer "F.Cu")
-		(name "$teardrop_padvia$")
-		(hatch none 0.1)
-		(priority 30001)
-		(attr
-			(teardrop
-				(type padvia)
-			)
-		)
-		(connect_pads yes
-			(clearance 0)
-		)
-		(min_thickness 0.0254)
-		(filled_areas_thickness no)
-		(fill yes
-			(thermal_gap 0.5)
-			(thermal_bridge_width 0.5)
-			(island_removal_mode 1)
-			(island_area_min 10)
-		)
-		(polygon
-			(pts
-				(xy 166.724 76.974169) (xy 166.524 76.974169) (xy 165.991075 78.04308) (xy 166.614677 79.910758)
-				(xy 167.238279 78.04308)
-			)
-		)
